Commit message: gazebo所有的设备雷达点云等都已经设置正确。

File: bot_description/urdf/lekiwi_bot.gazebo.xacro (robot description, xacro)
@@ -31,9 +31,15 @@
   </gazebo>
   <!-- RGB-D 相机插件 (模拟Astra Pro) -->
-  <gazebo reference="Camera-Model-v3">
+  <!--
+    重要说明：
+    - Gazebo 传感器附着在 camera_link（使用 Gazebo 相机约定：+X 看向前方）
+    - frame_name 设置为 camera_optical_frame（符合 ROS 光学坐标系约定）
+    - 这样 Gazebo 渲染正确，同时 ROS 消息使用正确的 frame
+  -->
+  <gazebo reference="camera_link">
     <sensor name="camera" type="depth">
       <update_rate>30</update_rate>
-      <camera>
-        <horizontal_fov>1.047</horizontal_fov>  <!-- 60度 -->
+      <camera name="camera">
+        <horizontal_fov>1.047</horizontal_fov>
         <image>
           <width>640</width>
@@ -42,22 +48,23 @@
         </image>
         <clip>
-          <near>0.6</near>
+          <near>0.05</near>
           <far>8.0</far>
         </clip>
+        <noise>
+          <type>gaussian</type>
+          <mean>0.0</mean>
+          <stddev>0.007</stddev>
+        </noise>
       </camera>
       <plugin name="camera_controller" filename="libgazebo_ros_camera.so">
         <camera_name>camera</camera_name>
-        <frame_name>Camera-Model-v3</frame_name>
-        <!-- 话题命名 -->
-        <image_topic>color/image_raw</image_topic>
-        <camera_info_topic>color/camera_info</camera_info_topic>
-        <depth_image_topic>depth/image_raw</depth_image_topic>
-        <depth_image_camera_info_topic>depth/camera_info</depth_image_camera_info_topic>
-        <point_cloud_topic>depth/points</point_cloud_topic>
-        <!-- 深度相机参数 -->
-        <min_depth>0.6</min_depth>
-        <max_depth>8.0</max_depth>
+        <frame_name>camera_optical_frame</frame_name>
+        <hack_baseline>0.07</hack_baseline>
       </plugin>
     </sensor>
+  </gazebo>
+  <!-- Camera-Model-v3 材质 -->
+  <gazebo reference="Camera-Model-v3">
+    <material>Gazebo/Black</material>
   </gazebo>
   <!-- 材质颜色定义 -->
@@ -103,7 +110,3 @@
     <material>Gazebo/Orange</material>
   </gazebo>
-  <!-- 相机 -->
-  <gazebo reference="Camera-Model-v3">
-    <material>Gazebo/Black</material>
-  </gazebo>
 </robot>

File: bot_description/urdf/lekiwi_bot.xacro (robot description, xacro)
@@ -16,4 +16,5 @@
     <xacro:property name="M_PI_6" value="0.5235987755982988" />    <!-- π/6 = 30° -->
     <xacro:property name="DEG_15" value="0.26179938779914924" />   <!-- 15° -->
+    <xacro:property name="DEG_10" value="0.17453292519943295" />   <!-- 10° -->
     <xacro:property name="DEG_75" value="1.3089969389957468" />    <!-- 75° -->
     <xacro:property name="DEG_80" value="1.3962634015954636" />    <!-- 80° -->
@@ -439,4 +440,55 @@
         <child link="Camera-Model-v3" />
     </joint>
+    <!--
+        相机坐标系（双 Frame 结构）/ Camera Frames (Dual Frame Structure)
+        说明 / Description:
+        1. camera_link: Gazebo 传感器附着点，使用 Gazebo 相机约定
+           - Gazebo 相机看向 +X 方向，图像上方是 +Z
+           - 此 frame 与 base_link 方向相同，位于镜头前方
+        2. camera_optical_frame: ROS 光学坐标系约定
+           - Z 轴是光轴（指向前方），Y 轴是图像下方，X 轴是图像右方
+           - 用于点云、深度图像等 ROS 数据处理
+    -->
+    <!-- camera_link: Gazebo 传感器使用此 frame -->
+    <link name="camera_link">
+        <!-- 空 link，仅用作 Gazebo 传感器附着点 -->
+    </link>
+    <!-- Camera-Model-v3 -> camera_link -->
+    <joint name="camera_link_joint" type="fixed">
+        <!--
+            目标: camera_link 在 base_link 中位于 [0.146, 0, 0.038]，方向与 base_link 相同
+            这样 Gazebo 相机会看向机器人前方(+X)，横屏显示
+            计算: T_joint = T_base_cam_model^(-1) @ T_base_cam_link
+            其中 T_base_cam_model 来自 tf2_echo
+        -->
+        <origin xyz="-0.002425 0.040000 -0.013788" rpy="${DEG_100} 0 ${M_PI_2}" />
+        <parent link="Camera-Model-v3" />
+        <child link="camera_link" />
+    </joint>
+    <!-- camera_optical_frame: ROS 光学坐标系 -->
+    <link name="camera_optical_frame">
+        <!-- 空 link，仅用作光学坐标系参考 -->
+    </link>
+    <!-- camera_link -> camera_optical_frame -->
+    <joint name="camera_optical_frame_joint" type="fixed">
+        <!--
+            标准的 Gazebo -> ROS 光学坐标系转换
+            从 Gazebo 约定 (X前, Y左, Z上) 到 ROS 光学约定 (Z前, X右, Y下)
+            旋转: 先绕 Y 轴 -90° (X->Z)，再绕 X 轴 -90° (Y->-Z, Z->Y)
+            等效 RPY: [-π/2, 0, -π/2]
+        -->
+        <origin xyz="0 0 0" rpy="-${M_PI_2} 0 -${M_PI_2}" />
+        <parent link="camera_link" />
+        <child link="camera_optical_frame" />
+    </joint>
+    <!-- 兼容性别名: camera_frame 指向 camera_optical_frame -->
+    <link name="camera_frame">
+        <!-- 保持向后兼容 -->
+    </link>
+    <joint name="camera_frame_joint" type="fixed">
+        <origin xyz="0 0 0" rpy="0 0 0" />
+        <parent link="camera_optical_frame" />
+        <child link="camera_frame" />
+    </joint>
     <!-- ====================================================================== -->
     <!-- 第7部分: 支撑铜柱与第二层底板 / Part 7: Standoffs and Second Layer     -->
