Commit message: 临时提交一下修正后的urdf

File: bot_description/urdf/lekiwi_bot.gazebo.xacro (robot description, xacro)
@@ -6,13 +6,15 @@
   <!-- 用于 LeKiwi 三轮全向机器人的 Gazebo 仿真                                -->
   <!-- ====================================================================== -->
+  <!-- Controller configuration file path / 控制器配置文件路径 -->
+  <xacro:arg name="controller_config_file" default="$(find bot_control)/config/omni_wheel_controller.yaml"/>
   <!-- ====================================================================== -->
   <!-- Xacro Arguments / Xacro 参数                                            -->
   <!-- ====================================================================== -->
   <!--
-    publish_odom_tf: Control whether Gazebo publishes odom->base_link TF
+    publish_odom_tf - Control whether Gazebo publishes odom->base_link TF
     发布里程计 TF：控制 Gazebo 是否发布 odom->base_link TF 变换
-    - true (default): Gazebo publishes TF, suitable for basic simulation
+    - true (default) - Gazebo publishes TF, suitable for basic simulation
     - true（默认）：Gazebo 发布 TF，适用于基本仿真
-    - false: Disable TF publishing, required when using external odometry fusion
+    - false - Disable TF publishing, required when using external odometry fusion
              (e.g., robot_localization EKF with visual odometry)
     - false：禁用 TF 发布，当使用外部里程计融合时需要
@@ -21,44 +23,14 @@
   <xacro:arg name="publish_odom_tf" default="true"/>
   <!-- ====================================================================== -->
-  <!-- Omnidirectional Wheel Motion Plugin (Planar Move)                      -->
-  <!-- 全向轮移动插件 (Planar Move)                                            -->
+  <!-- ros2_control Gazebo Plugin                                             -->
+  <!-- ros2_control Gazebo 插件                                                -->
+  <!-- Hardware-level wheel simulation replacing planar_move                  -->
+  <!-- 硬件级轮子仿真替代planar_move                                           -->
   <!-- ====================================================================== -->
   <gazebo>
-    <plugin name="omni_drive_controller" filename="libgazebo_ros_planar_move.so">
-      <!-- Update Rate / 更新频率 -->
-      <update_rate>50.0</update_rate>
-      <!-- Command Topic / 命令话题 -->
-      <command_topic>cmd_vel</command_topic>
-      <!-- Odometry Topic / 里程计话题 -->
-      <odometry_topic>odom</odometry_topic>
-      <!-- Frame Configuration / 坐标系配置 -->
-      <odometry_frame>odom</odometry_frame>
-      <robot_base_frame>base_link</robot_base_frame>
-      <!--
-        Odometry Publishing Configuration / 里程计发布配置
-        publish_odom: Always publish odometry messages
-        publish_odom_tf: Controlled by xacro arg for VIO compatibility
-        publish_odom：始终发布里程计消息
-        publish_odom_tf：由 xacro 参数控制以兼容 VIO
-      -->
-      <publish_odom>true</publish_odom>
-      <publish_odom_tf>$(arg publish_odom_tf)</publish_odom_tf>
-      <!-- Velocity Limits / 速度限制 -->
-      <!-- 提高速度限制以加快导航测试 / Increase velocity for faster navigation -->
-      <max_vel_x>0.35</max_vel_x>
-      <max_vel_y>0.35</max_vel_y>
-      <max_vel_yaw>2.0</max_vel_yaw>
-      <!--
-        Covariance Configuration / 协方差配置
-        These values represent the uncertainty in wheel odometry
-        这些值表示轮式里程计的不确定性
-      -->
-      <covariance_x>0.0001</covariance_x>
-      <covariance_y>0.0001</covariance_y>
-      <covariance_yaw>0.01</covariance_yaw>
-      <!-- Velocity decay when no command / 无命令时速度衰减 -->
-      <!-- Timeout after which robot stops if no cmd_vel received -->
-      <!-- 接收不到cmd_vel命令后机器人停止的超时时间 -->
-      <cmd_timeout>0.5</cmd_timeout>
+    <plugin filename="libgazebo_ros2_control.so" name="gazebo_ros2_control">
+      <!-- Controller configuration file -->
+      <!-- xacro will substitute $(arg xxx) before Gazebo sees it -->
+      <parameters>$(arg controller_config_file)</parameters>
     </plugin>
   </gazebo>
@@ -101,5 +73,5 @@
         <min_depth>0.10</min_depth>
         <max_depth>6.0</max_depth>
-        <!-- 关键优化:将cutoff设为极小值 / Key optimization: set cutoff to minimal value -->
+        <!-- 关键优化 将cutoff设为极小值 / Key optimization set cutoff to minimal value -->
         <!-- 只保留0.03米内的点(实际上几乎没有),避免靠墙时触发大量点云计算 -->
         <!-- Only keep points within 0.03m (virtually none), avoid massive point cloud when near walls -->
@@ -119,30 +91,41 @@
     <material>Gazebo/White</material>
   </gazebo>
+  <!-- 左前轮物理属性 / Left Front Wheel Physics (suffix="") -->
   <gazebo reference="4-Omni-Directional-Wheel_Single_Body-v1">
     <material>Gazebo/Black</material>
-    <mu1>0.1</mu1>
-    <mu2>0.1</mu2>
+    <!-- mu1 lateral friction, mu2 rolling friction -->
+    <mu1>0.8</mu1>
+    <mu2>0.01</mu2>
+    <!-- slip1/slip2 - omnidirectional wheel behavior -->
+    <slip1>0.1</slip1>
+    <slip2>0.9</slip2>
     <kp>1000000.0</kp>
     <kd>100.0</kd>
     <minDepth>0.001</minDepth>
-    <maxVel>1.0</maxVel>
+    <maxVel>10.0</maxVel>
   </gazebo>
+  <!-- 右前轮物理属性 / Right Front Wheel Physics (suffix="-1") -->
   <gazebo reference="4-Omni-Directional-Wheel_Single_Body-v1-1">
     <material>Gazebo/Black</material>
-    <mu1>0.1</mu1>
-    <mu2>0.1</mu2>
+    <mu1>0.8</mu1>
+    <mu2>0.01</mu2>
+    <slip1>0.1</slip1>
+    <slip2>0.9</slip2>
     <kp>1000000.0</kp>
     <kd>100.0</kd>
     <minDepth>0.001</minDepth>
-    <maxVel>1.0</maxVel>
+    <maxVel>10.0</maxVel>
   </gazebo>
+  <!-- 后轮物理属性 / Rear Wheel Physics (suffix="-2") -->
   <gazebo reference="4-Omni-Directional-Wheel_Single_Body-v1-2">
     <material>Gazebo/Black</material>
-    <mu1>0.1</mu1>
-    <mu2>0.1</mu2>
+    <mu1>0.8</mu1>
+    <mu2>0.01</mu2>
+    <slip1>0.1</slip1>
+    <slip2>0.9</slip2>
     <kp>1000000.0</kp>
     <kd>100.0</kd>
     <minDepth>0.001</minDepth>
-    <maxVel>1.0</maxVel>
+    <maxVel>10.0</maxVel>
   </gazebo>
   <!-- 电池 -->

File: bot_description/urdf/lekiwi_bot.xacro (robot description, xacro)
@@ -2,5 +2,5 @@
 <robot xmlns:xacro="http://www.ros.org/wiki/xacro" name="LeKiwi">
     <!-- ====================================================================== -->
-    <!-- 第1部分: 常量与属性定义 / Part 1: Constants and Properties             -->
+    <!-- 第1部分- 常量与属性定义 / Part 1- Constants and Properties             -->
     <!-- ====================================================================== -->
     <material name="White">
@@ -26,5 +26,5 @@
     <xacro:property name="mesh_scale" value="0.001 0.001 0.001" />
     <!-- ====================================================================== -->
-    <!-- 第2部分: 宏定义 / Part 2: Macro Definitions                            -->
+    <!-- 第2部分- 宏定义 / Part 2- Macro Definitions                            -->
     <!-- ====================================================================== -->
     <!--
@@ -32,5 +32,5 @@
         用于创建包含惯性、视觉和碰撞属性的 link
         Used to create links with inertial, visual, and collision properties
-        参数 material_name: 材质颜色名称，默认为 White / Material color name, default is White
+        参数 material_name- 材质颜色名称，默认为 White / Material color name- default is White
     -->
     <xacro:macro name="mesh_link"
@@ -85,6 +85,6 @@
     <!--
         轮组装配宏 / Wheel Assembly Macro
-        包含: 电机支架 -> 舵机 -> 轮毂 -> 全向轮
-        Contains: Motor Mount -> Servo Motor -> Wheel Mount -> Omni Wheel
+        包含- 电机支架 -> 舵机 -> 轮毂 -> 全向轮
+        Contains- Motor Mount -> Servo Motor -> Wheel Mount -> Omni Wheel
     -->
     <xacro:macro name="wheel_assembly"
@@ -162,12 +162,14 @@
             material_name="Black" />
         <!-- 轮毂到全向轮的关节 / Joint from Wheel Mount to Omni Wheel -->
-        <joint name="omni_wheel_mount-v5${suffix}_to_wheel" type="fixed">
+        <joint name="omni_wheel_mount-v5${suffix}_to_wheel" type="continuous">
             <origin xyz="${wheel_joint_xyz}" rpy="${wheel_joint_rpy}" />
             <parent link="omni_wheel_mount-v5${suffix}" />
             <child link="4-Omni-Directional-Wheel_Single_Body-v1${suffix}" />
+            <axis xyz="${wheel_axis}" />
+            <dynamics damping="0.1" friction="0.1"/>
         </joint>
     </xacro:macro>
     <!-- ====================================================================== -->
-    <!-- 第3部分: 底盘基座 / Par    source ~/.bashrc    source ~/.bashrct 3: Chassis Base                               -->
+    <!-- 第3部分- 底盘基座 / Part 3- Chassis Base                               -->
     <!-- ====================================================================== -->
     <!--
@@ -194,8 +196,8 @@
     </joint>
     <!-- ====================================================================== -->
-    <!-- 第4部分: 轮组装配 (3组全向轮) / Part 4: Wheel Assemblies (3 Omni Wheels) -->
-    <!-- ====================================================================== -->
-    <!--
-        轮组1: 后轮 (Back Wheel) - suffix: -2
+    <!-- 第4部分- 轮组装配 (3组全向轮) / Part 4- Wheel Assemblies (3 Omni Wheels) -->
+    <!-- ====================================================================== -->
+    <!--
+        轮组1- 后轮 (Back Wheel) - suffix- -2
         base_plate_layer1 -> drive_motor_mount-2 -> servo_motor-2 -> wheel_mount-2 -> wheel-2
     -->
@@ -248,5 +250,5 @@
         wheel_visual_rpy="${M_PI_2} ${DEG_15} 0" />
     <!--
-        轮组2: 右前轮 (Right Front Wheel) - suffix: -1
+        轮组2- 右前轮 (Right Front Wheel) - suffix- -1
         base_plate_layer1 -> drive_motor_mount-1 -> servo_motor-1 -> wheel_mount-1 -> wheel-1
     -->
@@ -299,5 +301,5 @@
         wheel_visual_rpy="-${M_PI_6} -${M_PI_2} 0" />
     <!--
-        轮组3: 左前轮 (Left Front Wheel) - suffix: (empty)
+        轮组3- 左前轮 (Left Front Wheel) - suffix- (empty)
         base_plate_layer1 -> drive_motor_mount -> servo_motor -> wheel_mount -> wheel
     -->
@@ -350,5 +352,5 @@
         wheel_visual_rpy="${M_PI_2} -${DEG_75} ${DEG_120}" />
     <!-- ====================================================================== -->
-    <!-- 第5部分: 电子元器件 / Part 5: Electronic Components                    -->
+    <!-- 第5部分- 电子元器件 / Part 5- Electronic Components                    -->
     <!-- ====================================================================== -->
     <!-- 舵机控制器支架 / Servo Controller Mount -->
@@ -404,5 +406,5 @@
     </joint>
     <!-- ====================================================================== -->
-    <!-- 第6部分: 相机系统 / Part 6: Camera System                              -->
+    <!-- 第6部分- 相机系统 / Part 6- Camera System                              -->
     <!-- ====================================================================== -->
     <!-- 相机支架 / Camera Mount -->
@@ -442,13 +444,13 @@
     <!--
         相机坐标系（双 Frame 结构）/ Camera Frames (Dual Frame Structure)
-        说明 / Description:
-        1. camera_link: Gazebo 传感器附着点，使用 Gazebo 相机约定
+        说明 / Description-
+        1. camera_link- Gazebo 传感器附着点，使用 Gazebo 相机约定
            - Gazebo 相机看向 +X 方向，图像上方是 +Z
            - 此 frame 与 base_link 方向相同，位于镜头前方
-        2. camera_optical_frame: ROS 光学坐标系约定
+        2. camera_optical_frame- ROS 光学坐标系约定
            - Z 轴是光轴（指向前方），Y 轴是图像下方，X 轴是图像右方
            - 用于点云、深度图像等 ROS 数据处理
     -->
-    <!-- camera_link: Gazebo 传感器使用此 frame -->
+    <!-- camera_link- Gazebo 传感器使用此 frame -->
     <link name="camera_link">
         <!-- 空 link，仅用作 Gazebo 传感器附着点 -->
@@ -457,7 +459,7 @@
     <joint name="camera_link_joint" type="fixed">
         <!--
-            目标: camera_link 在 base_link 中位于 [0.146, 0, 0.038]，方向与 base_link 相同
+            目标- camera_link 在 base_link 中位于 [0.146, 0, 0.038]，方向与 base_link 相同
             这样 Gazebo 相机会看向机器人前方(+X)，横屏显示
-            计算: T_joint = T_base_cam_model^(-1) @ T_base_cam_link
+            计算- T_joint = T_base_cam_model^(-1) @ T_base_cam_link
             其中 T_base_cam_model 来自 tf2_echo
         -->
@@ -466,5 +468,5 @@
         <child link="camera_link" />
     </joint>
-    <!-- camera_optical_frame: ROS 光学坐标系 -->
+    <!-- camera_optical_frame- ROS 光学坐标系 -->
     <link name="camera_optical_frame">
         <!-- 空 link，仅用作光学坐标系参考 -->
@@ -475,6 +477,6 @@
             标准的 Gazebo -> ROS 光学坐标系转换
             从 Gazebo 约定 (X前, Y左, Z上) 到 ROS 光学约定 (Z前, X右, Y下)
-            旋转: 先绕 Y 轴 -90° (X->Z)，再绕 X 轴 -90° (Y->-Z, Z->Y)
-            等效 RPY: [-π/2, 0, -π/2]
+            旋转- 先绕 Y 轴 -90° (X->Z)，再绕 X 轴 -90° (Y->-Z, Z->Y)
+            等效 RPY- [-π/2, 0, -π/2]
         -->
         <origin xyz="0 0 0" rpy="-${M_PI_2} 0 -${M_PI_2}" />
@@ -482,5 +484,5 @@
         <child link="camera_optical_frame" />
     </joint>
-    <!-- 兼容性别名: camera_frame 指向 camera_optical_frame -->
+    <!-- 兼容性别名- camera_frame 指向 camera_optical_frame -->
     <link name="camera_frame">
         <!-- 保持向后兼容 -->
@@ -492,5 +494,5 @@
     </joint>
     <!-- ====================================================================== -->
-    <!-- 第7部分: 支撑铜柱与第二层底板 / Part 7: Standoffs and Second Layer     -->
+    <!-- 第7部分- 支撑铜柱与第二层底板 / Part 7- Standoffs and Second Layer     -->
     <!-- ====================================================================== -->
     <!--
@@ -498,5 +500,5 @@
         连接底板第一层和第二层 / Connect base plate layer 1 and layer 2
     -->
-    <!-- 铜柱0: 中心 / Standoff 0: Center -->
+    <!-- 铜柱0- 中心 / Standoff 0- Center -->
     <xacro:hex_standoff suffix=""
         mesh_file="94868A713_NO-THREADS_Female-Threaded-Hex-Standoff.stl"
@@ -506,5 +508,5 @@
         inertial_z="-0.02499999330297986"
         visual_z="-0.025" />
-    <!-- 铜柱1: 左侧 / Standoff 1: Left -->
+    <!-- 铜柱1- 左侧 / Standoff 1- Left -->
     <xacro:hex_standoff suffix="-1"
         mesh_file="94868A713_NO-THREADS_Female-Threaded-Hex-Standoff-1.stl"
@@ -514,5 +516,5 @@
         inertial_z="-0.02499999330297986"
         visual_z="-0.025" />
-    <!-- 铜柱2: 右侧 / Standoff 2: Right -->
+    <!-- 铜柱2- 右侧 / Standoff 2- Right -->
     <xacro:hex_standoff suffix="-2"
         mesh_file="94868A713_NO-THREADS_Female-Threaded-Hex-Standoff-2.stl"
@@ -522,5 +524,5 @@
         inertial_z="-0.02481596290467566"
         visual_z="-0.0248159696016958" />
-    <!-- 铜柱3: 左后 / Standoff 3: Left Rear -->
+    <!-- 铜柱3- 左后 / Standoff 3- Left Rear -->
     <xacro:hex_standoff suffix="-3"
         mesh_file="94868A713_NO-THREADS_Female-Threaded-Hex-Standoff-3.stl"
@@ -530,5 +532,5 @@
         inertial_z="-0.024999993302979855"
         visual_z="-0.025" />
-    <!-- 铜柱4: 右后 / Standoff 4: Right Rear -->
+    <!-- 铜柱4- 右后 / Standoff 4- Right Rear -->
     <xacro:hex_standoff suffix="-4"
         mesh_file="94868A713_NO-THREADS_Female-Threaded-Hex-Standoff-4.stl"
@@ -538,5 +540,5 @@
         inertial_z="-0.02499999330297986"
         visual_z="-0.025" />
-    <!-- 铜柱5: 前方 / Standoff 5: Front -->
+    <!-- 铜柱5- 前方 / Standoff 5- Front -->
     <xacro:hex_standoff suffix="-5"
         mesh_file="94868A713_NO-THREADS_Female-Threaded-Hex-Standoff-5.stl"
@@ -564,5 +566,5 @@
     </joint>
     <!-- ====================================================================== -->
-    <!-- 第8部分: 顶部盖板 / Part 8: Top Covers                                 -->
+    <!-- 第8部分- 顶部盖板 / Part 8- Top Covers                                 -->
     <!-- ====================================================================== -->
     <!-- 底部盖板 / Bottom Cover -->
@@ -600,3 +602,38 @@
         <child link="Top-V2-v2" />
     </joint>
+    <!-- ====================================================================== -->
+    <!-- ros2_control Configuration                                             -->
+    <!-- ====================================================================== -->
+    <ros2_control name="GazeboSystem" type="system">
+        <hardware>
+            <plugin>gazebo_ros2_control/GazeboSystem</plugin>
+        </hardware>
+        <!-- Wheel 1 Rear -->
+        <joint name="omni_wheel_mount-v5-2_to_wheel">
+            <command_interface name="velocity">
+                <param name="min">-100</param>
+                <param name="max">100</param>
+            </command_interface>
+            <state_interface name="position"/>
+            <state_interface name="velocity"/>
+        </joint>
+        <!-- Wheel 2 Right Front -->
+        <joint name="omni_wheel_mount-v5-1_to_wheel">
+            <command_interface name="velocity">
+                <param name="min">-100</param>
+                <param name="max">100</param>
+            </command_interface>
+            <state_interface name="position"/>
+            <state_interface name="velocity"/>
+        </joint>
+        <!-- Wheel 3 Left Front -->
+        <joint name="omni_wheel_mount-v5_to_wheel">
+            <command_interface name="velocity">
+                <param name="min">-100</param>
+                <param name="max">100</param>
+            </command_interface>
+            <state_interface name="position"/>
+            <state_interface name="velocity"/>
+        </joint>
+    </ros2_control>
 </robot>

File: bot_description/urdf/lekiwi_bot_imu.gazebo.xacro (robot description, xacro)
@@ -10,6 +10,6 @@
     <!-- ====================================================================== -->
     <!--
-        Issue: Gazebo IMU on imu_link with low mass causes unstable physics
-        Solution: Use gravity and orientation only, minimal noise
+        Issue - Gazebo IMU on imu_link with low mass causes unstable physics
+        Solution - Use gravity and orientation only, minimal noise
         问题：imu_link质量太小导致Gazebo IMU物理计算不稳定
         解决：只使用重力和方向，最小化噪声
@@ -21,4 +21,22 @@
             <update_rate>100</update_rate>
             <visualize>false</visualize>
+            <!-- IMU Noise Model / IMU 噪声模型 -->
+            <!-- Required by Gazebo to avoid "Get noise index not valid" errors -->
+            <!-- Gazebo 要求定义噪声模型以避免 "Get noise index not valid" 错误 -->
+            <imu>
+                <noise>
+                    <!-- Angular velocity noise (rad/s) / 角速度噪声 -->
+                    <type>gaussian</type>
+                    <rate>
+                        <mean>0.0</mean>
+                        <stddev>0.001</stddev>
+                    </rate>
+                    <!-- Linear acceleration noise (m/s^2) / 线性加速度噪声 -->
+                    <accel>
+                        <mean>0.0</mean>
+                        <stddev>0.01</stddev>
+                    </accel>
+                </noise>
+            </imu>
             <plugin name="imu_plugin" filename="libgazebo_ros_imu_sensor.so">
                 <ros>

Commit message: 现在终于将三个轮子的旋转都正常了，需要调整gazebo 的测试模拟数据，保证模拟机器人的运动。

File: bot_description/urdf/lekiwi_bot.gazebo.xacro (robot description, xacro)
@@ -95,11 +95,11 @@
     <material>Gazebo/Black</material>
     <!-- mu1 lateral friction, mu2 rolling friction -->
-    <mu1>0.8</mu1>
-    <mu2>0.01</mu2>
+    <mu1>1.0</mu1>
+    <mu2>0.5</mu2>
     <!-- slip1/slip2 - omnidirectional wheel behavior -->
-    <slip1>0.1</slip1>
-    <slip2>0.9</slip2>
+    <slip1>0.5</slip1>
+    <slip2>0.5</slip2>
     <kp>1000000.0</kp>
-    <kd>100.0</kd>
+    <kd>10.0</kd>
     <minDepth>0.001</minDepth>
     <maxVel>10.0</maxVel>
@@ -108,10 +108,10 @@
   <gazebo reference="4-Omni-Directional-Wheel_Single_Body-v1-1">
     <material>Gazebo/Black</material>
-    <mu1>0.8</mu1>
-    <mu2>0.01</mu2>
-    <slip1>0.1</slip1>
-    <slip2>0.9</slip2>
+    <mu1>1.0</mu1>
+    <mu2>0.5</mu2>
+    <slip1>0.5</slip1>
+    <slip2>0.5</slip2>
     <kp>1000000.0</kp>
-    <kd>100.0</kd>
+    <kd>10.0</kd>
     <minDepth>0.001</minDepth>
     <maxVel>10.0</maxVel>
@@ -120,10 +120,10 @@
   <gazebo reference="4-Omni-Directional-Wheel_Single_Body-v1-2">
     <material>Gazebo/Black</material>
-    <mu1>0.8</mu1>
-    <mu2>0.01</mu2>
-    <slip1>0.1</slip1>
-    <slip2>0.9</slip2>
+    <mu1>1.0</mu1>
+    <mu2>0.5</mu2>
+    <slip1>0.5</slip1>
+    <slip2>0.5</slip2>
     <kp>1000000.0</kp>
-    <kd>100.0</kd>
+    <kd>10.0</kd>
     <minDepth>0.001</minDepth>
     <maxVel>10.0</maxVel>

File: bot_description/urdf/lekiwi_bot.xacro (robot description, xacro)
@@ -167,5 +167,5 @@
             <child link="4-Omni-Directional-Wheel_Single_Body-v1${suffix}" />
             <axis xyz="${wheel_axis}" />
-            <dynamics damping="0.1" friction="0.1"/>
+            <dynamics damping="0.001" friction="0.001"/>
         </joint>
     </xacro:macro>
@@ -230,5 +230,5 @@
         wheel_revolute_xyz="0.01025 -0.0352 -0.03275"
         wheel_revolute_rpy="-${M_PI_2} ${M_PI_2} 0"
-        wheel_axis="0 0 -1.0"
+        wheel_axis="0 1.0 0"
         wheel_mount_inertial_xyz="0 0 -0.005522899140934374"
         wheel_mount_inertial_rpy="0 0 0"
@@ -281,5 +281,5 @@
         wheel_revolute_xyz="0.01025 0.04636234 -0.01480191"
         wheel_revolute_rpy="-${M_PI_2} ${M_PI_2} 0"
-        wheel_axis="0.866025 0 0.5"
+        wheel_axis="-0.866025 0.5 0"
         wheel_mount_inertial_xyz="0.004782968825905343 0 0.0027614494161754166"
         wheel_mount_inertial_rpy="0 0 0"
@@ -332,5 +332,5 @@
         wheel_revolute_xyz="0.01025 -0.01076234 0.04685909"
         wheel_revolute_rpy="-${M_PI_2} ${M_PI_2} 0"
-        wheel_axis="-0.866025 0 0.5"
+        wheel_axis="-0.866025 -0.5 0"
         wheel_mount_inertial_xyz="-0.00478297352513172 0 0.002761449724759064"
         wheel_mount_inertial_rpy="0 0 0"
