Commit message: 调整了物理属性，基本可以直行，还是要微调

File: bot_description/urdf/lekiwi_bot.gazebo.xacro (robot description, xacro)
@@ -31,6 +31,6 @@
     <plugin filename="libgazebo_ros2_control.so" name="gazebo_ros2_control">
       <!-- Controller configuration file -->
-      <!-- xacro will substitute $(arg xxx) before Gazebo sees it -->
       <parameters>$(arg controller_config_file)</parameters>
+      <!-- PID gains are now loaded from gazebo_pid_gains.yaml -->
     </plugin>
   </gazebo>
@@ -96,11 +96,11 @@
     <!-- 全向轮关键参数：高滚动摩擦 + 极低侧向摩擦 -->
     <mu1>2.0</mu1>      <!-- 滚动摩擦系数-提供足够抓地力（增加到2.0） -->
-    <mu2>0.0</mu2>      <!-- 侧向摩擦系数-设为0允许完全自由滑动 -->
+    <mu2>0.1</mu2>      <!-- 侧向摩擦系数-轻微摩擦提供稳定性 -->
     <kp>10000000.0</kp> <!-- 接触刚度-提高10倍避免轮子下沉 -->
     <kd>1.0</kd>        <!-- 接触阻尼-降低减少能量损失 -->
     <minDepth>0.0001</minDepth>  <!-- 最小接触深度 -->
     <maxVel>100.0</maxVel>
-    <!-- 添加滚动阻力参数 -->
-    <fdir1>1 0 0</fdir1>  <!-- 第一摩擦方向（滚动方向） -->
+    <!-- 第一摩擦方向=轮子axis方向 (与URDF中axis="0.866025 0.5 0"一致) -->
+    <fdir1>0.866025 0.5 0</fdir1>
   </gazebo>
   <!-- 右前轮物理属性 / Right Front Wheel Physics (suffix="-1") -->
@@ -108,10 +108,11 @@
     <material>Gazebo/Black</material>
     <mu1>2.0</mu1>
-    <mu2>0.0</mu2>
+    <mu2>0.1</mu2>
     <kp>10000000.0</kp>
     <kd>1.0</kd>
     <minDepth>0.0001</minDepth>
     <maxVel>100.0</maxVel>
-    <fdir1>1 0 0</fdir1>
+    <!-- 第一摩擦方向=轮子axis方向 (与URDF中axis="0.866025 -0.5 0"一致) -->
+    <fdir1>0.866025 -0.5 0</fdir1>
   </gazebo>
   <!-- 后轮物理属性 / Rear Wheel Physics (suffix="-2") -->
@@ -119,10 +120,11 @@
     <material>Gazebo/Black</material>
     <mu1>2.0</mu1>
-    <mu2>0.0</mu2>
+    <mu2>0.1</mu2>
     <kp>10000000.0</kp>
     <kd>1.0</kd>
     <minDepth>0.0001</minDepth>
     <maxVel>100.0</maxVel>
-    <fdir1>1 0 0</fdir1>
+    <!-- 第一摩擦方向=轮子axis方向 (与URDF中axis="0 -1.0 0"一致) -->
+    <fdir1>0 -1 0</fdir1>
   </gazebo>
   <!-- 电池 -->

File: bot_description/urdf/lekiwi_bot.xacro (robot description, xacro)
@@ -153,13 +153,27 @@
         </joint>
         <!-- 全向轮 Link / Omni Wheel Link -->
-        <xacro:mesh_link
-            name="4-Omni-Directional-Wheel_Single_Body-v1${suffix}"
-            mesh_file="${wheel_mesh}"
-            inertial_xyz="${wheel_inertial_xyz}" inertial_rpy="${wheel_inertial_rpy}"
-            mass="${wheel_mass}"
-            ixx="${wheel_ixx}" iyy="${wheel_iyy}" izz="${wheel_izz}"
-            ixy="${wheel_ixy}" iyz="${wheel_iyz}" ixz="${wheel_ixz}"
-            visual_xyz="${wheel_visual_xyz}" visual_rpy="${wheel_visual_rpy}"
-            material_name="Black" />
+        <link name="4-Omni-Directional-Wheel_Single_Body-v1${suffix}">
+            <inertial>
+                <origin xyz="${wheel_inertial_xyz}" rpy="${wheel_inertial_rpy}" />
+                <mass value="${wheel_mass}" />
+                <inertia ixx="${wheel_ixx}" iyy="${wheel_iyy}" izz="${wheel_izz}"
+                    ixy="${wheel_ixy}" iyz="${wheel_iyz}" ixz="${wheel_ixz}" />
+            </inertial>
+            <visual name="4-Omni-Directional-Wheel_Single_Body-v1${suffix}_visual">
+                <origin xyz="${wheel_visual_xyz}" rpy="${wheel_visual_rpy}" />
+                <geometry>
+                    <mesh filename="${mesh_pkg}/${wheel_mesh}" scale="${mesh_scale}" />
+                </geometry>
+                <material name="Black" />
+            </visual>
+            <!-- 简化碰撞体：使用圆柱体代替复杂mesh，确保物理计算准确 -->
+            <collision name="4-Omni-Directional-Wheel_Single_Body-v1${suffix}_collision">
+                <origin xyz="0 0 0" rpy="0 0 0" />
+                <geometry>
+                    <!-- 轮子直径0.1m(半径0.05m)，宽度0.032m -->
+                    <cylinder radius="0.05" length="0.032"/>
+                </geometry>
+            </collision>
+        </link>
         <!-- 轮毂到全向轮的关节 / Joint from Wheel Mount to Omni Wheel -->
         <!-- 主动驱动关节 - 轮子滚动，方向由机械结构固定 -->
@@ -169,5 +183,6 @@
             <child link="4-Omni-Directional-Wheel_Single_Body-v1${suffix}" />
             <axis xyz="${wheel_axis}" />
-            <dynamics damping="0.001" friction="0.001"/>
+            <!-- 极低damping确保速度响应快速，摩擦力由碰撞体mu1/mu2控制 -->
+            <dynamics damping="0.25" friction="0.001"/>
         </joint>
     </xacro:macro>
@@ -232,5 +247,5 @@
         wheel_revolute_xyz="0.01025 -0.0352 -0.03275"
         wheel_revolute_rpy="-${M_PI_2} ${M_PI_2} 0"
-        wheel_axis="0 1.0 0"
+        wheel_axis="0 -1.0 0"
         wheel_mount_inertial_xyz="0 0 -0.005522899140934374"
         wheel_mount_inertial_rpy="0 0 0"
@@ -283,5 +298,5 @@
         wheel_revolute_xyz="0.01025 0.04636234 -0.01480191"
         wheel_revolute_rpy="-${M_PI_2} ${M_PI_2} 0"
-        wheel_axis="-0.866025 0.5 0"
+        wheel_axis="0.866025 -0.5 0"
         wheel_mount_inertial_xyz="0.004782968825905343 0 0.0027614494161754166"
         wheel_mount_inertial_rpy="0 0 0"
@@ -334,5 +349,5 @@
         wheel_revolute_xyz="0.01025 -0.01076234 0.04685909"
         wheel_revolute_rpy="-${M_PI_2} ${M_PI_2} 0"
-        wheel_axis="-0.866025 -0.5 0"
+        wheel_axis="0.866025 0.5 0"
         wheel_mount_inertial_xyz="-0.00478297352513172 0 0.002761449724759064"
         wheel_mount_inertial_rpy="0 0 0"
@@ -611,5 +626,5 @@
             <plugin>gazebo_ros2_control/GazeboSystem</plugin>
         </hardware>
-        <!-- 轮子滚动关节 - 主动驱动 -->
+        <!-- 轮子滚动关节 - 主动驱动 (回退到Velocity Control) -->
         <!-- Wheel 1 Rear -->
         <joint name="omni_wheel_mount-v5-2_to_wheel">
